File: WBC_transmitter/file5FA50440.sch (KiCad schematic (older format))
At the start: 4 parts, among them U4 PIC16F1933-I_SS, Y1 Crystal

Commit message: Started Routing
Connections:
- wire segments 26 -> 28
Changed lines of the file:
@@
 Text GLabel 3400 4650 0    50   Input ~ 0
 IND_CUR
+Wire Wire Line
+	7200 -2100 7200 -3500
+Wire Wire Line
+	7200 -3500 4200 -3500
 $EndSCHEMATC
