File: WBC_transmitter/_autosave-WBC_transmitter.kicad_pcb (KiCad board)
At the start: 2 copper layers, 91 parts, among them J1 Conn_01x03_Female, J2 Conn_01x02_Female, J3 Conn_01x05_Male, J4 Conn_01x03_Female, J5 Conn_01x03_Female, J6 Conn_01x01_Male, J7 Conn_01x01_Male, Q1 IRF740, Q2 IRF740, Q3 IRF740, Q4 IRF740, Q5 IRF740, Q6 IRF740, U1 IR2110, U2 IR2110, U3 IR2110, U4 PIC16F1933-I_SS, U5 TL082, Y1 Crystal

Commit message: Routing 80%
Parts:
- J1: footprint Connector_JST:JST_EH_B3B-EH-A_1x03_P2.50mm_Vertical -> Connector_JST:JST_NV_B03P-NV_1x03_P5.00mm_Vertical
- L1, L2: footprint Resistor_THT:R_Axial_DIN0922_L20.0mm_D9.0mm_P7.62mm_Vertical -> Connector_JST:JST_EH_B2B-EH-A_1x02_P2.50mm_Vertical
- moved C11 147.6 mm to (161.3, 64.8)
- moved C12 139.7 mm to (150.5, 65.3)
- moved Y1 139.7 mm to (150.3, 69.9)
- moved J6 131.9 mm to (102.9, 57.1)
- moved Q6 120.0 mm to (186.7, 133.3), turned to 180 degrees
- moved L2 117.4 mm to (123.2, 134.6), turned to 180 degrees
- moved Q4 113.7 mm to (138.4, 133.3), turned to 180 degrees
- moved C17 109.7 mm to (201.9, 135.9), turned to 180 degrees
- moved D14 98.1 mm to (207.0, 135.9)
- moved C5 93.6 mm to (132.1, 81.3)
- moved U5 93.5 mm to (223.5, 121.9), turned to 90 degrees
- moved R16 92.0 mm to (198.1, 113.0), turned to 270 degrees
- moved J2 90.4 mm to (174.0, 133.3), turned to 180 degrees
- moved R19 89.3 mm to (217.2, 129.5), turned to 180 degrees
- moved C19 89.1 mm to (215.9, 115.6), turned to 270 degrees
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Routing:
- net CUR_2: track 110.6 -> 350.1 mm, vias 0 -> 2
- net BO-L: track 44.7 -> 251.7 mm
- net +300V: track 0.00 -> 176.7 mm
- net (no net): track 1.97 -> 135.0 mm, vias 0 -> 2
- net +100V: track 0.00 -> 129.6 mm, vias 0 -> 2
- net INV-VS: track 15.8 -> 115.1 mm, vias 0 -> 3
- net BO-H: track 48.2 -> 129.2 mm
- net GRID_C_SEN: track 0.00 -> 61.4 mm
- net BU-VS: track 35.8 -> 96.5 mm, vias 0 -> 1
- net +5V: track 95.2 -> 151.6 mm
- net Net-(R16-Pad1): track 0.00 -> 51.6 mm
- net Net-(D1-Pad2): track 0.00 -> 49.1 mm
- net +2.5V: track 0.00 -> 47.5 mm
- net +400V: track 0.00 -> 46.1 mm
- net Net-(C16-Pad2): track 0.00 -> 36.0 mm
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Other:
- board outline added: 153.7 x 88.9 mm
