File: WBC_transmitter/WBC_transmitter.kicad_pcb (KiCad board)
At the start: 2 copper layers, 153.7 x 88.9 mm, 91 parts, among them J1 Conn_01x03_Female, J2 Conn_01x02_Female, J3 Conn_01x05_Male, J4 Conn_01x03_Female, J5 Conn_01x03_Female, J6 Conn_01x01_Male, J7 Conn_01x01_Male, Q1 IRF740, Q2 IRF740, Q3 IRF740, Q4 IRF740, Q5 IRF740, Q6 IRF740, U1 IR2110, U2 IR2110, U3 IR2110, U4 PIC16F1933-I_SS, U5 TL082, Y1 Crystal

Commit message: 3 unrouted
Routing:
- net (no net): track 135.0 -> 3.37 mm, vias 2 -> 0
- net GRID_V_SEN: track 80.9 -> 205.5 mm, vias 3 -> 6
- net BO-H: track 129.2 -> 211.4 mm, vias 2 -> 8
- net GRID_C_SEN: track 61.4 -> 142.3 mm, vias 0 -> 3
- net +5V: track 264.4 -> 339.0 mm, vias 7 -> 12
- net CUR_2: track 455.9 -> 517.2 mm, vias 6 -> 9
- net INV-H: track 124.8 -> 174.0 mm, vias 9 -> 10
- net INVERTER_PWM: track 0.00 -> 39.5 mm, vias 0 -> 1
- net BOOST_PWM_INV: track 0.00 -> 38.0 mm, vias 0 -> 2
- net BUCK_PWM_INV: track 0.00 -> 32.1 mm, vias 0 -> 3
- net INVERTER_PWM_INV: track 0.00 -> 22.7 mm, vias 0 -> 2
- net INV-L: track 159.4 -> 138.1 mm, vias 3 -> 4
- net IND_CUR: track 0.11 -> 17.0 mm, vias 0 -> 2
- net BOOST_PWM: track 39.5 -> 56.2 mm, vias 5 -> 7
- net Net-(C12-Pad1): track 4.68 -> 18.0 mm
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