File: WBC_transmitter/WBC_transmitter.sch (KiCad schematic (older format))
At the start: 53 parts, among them J1 Conn_01x03_Female, J2 Conn_01x02_Female, J3 Conn_01x05_Male, J4 Conn_01x03_Female, J5 Conn_01x03_Female, J6 Conn_01x01_Male, J7 Conn_01x01_Male, Q1 IRF740, Q2 IRF740, Q3 IRF740, Q4 IRF740, Q5 IRF740, Q6 IRF740, U1 IR2110, U2 IR2110, U3 IR2110

Commit message: Finished Placing
Parts:
- J1: footprint Connector_JST:JST_EH_B3B-EH-A_1x03_P2.50mm_Vertical -> Connector_JST:JST_NV_B03P-NV_1x03_P5.00mm_Vertical
- L1, L2: footprint Resistor_THT:R_Axial_DIN0922_L20.0mm_D9.0mm_P7.62mm_Vertical -> Connector_JST:JST_EH_B2B-EH-A_1x02_P2.50mm_Vertical
Changed lines of the file:
@@
 F 0 "L2" H 9350 1765 50  0000 C CNN
 F 1 "INDUCTOR" H 9350 1674 50  0000 C CNN
-F 2 "Resistor_THT:R_Axial_DIN0922_L20.0mm_D9.0mm_P7.62mm_Vertical" H 9350 1550 50  0001 C CNN
+F 2 "Connector_JST:JST_EH_B2B-EH-A_1x02_P2.50mm_Vertical" H 9350 1550 50  0001 C CNN
 F 3 "~" H 9350 1550 50  0001 C CNN
 	1    9350 1550
@@
 F 0 "L1" H 5100 1515 50  0000 C CNN
 F 1 "INDUCTOR" H 5100 1424 50  0000 C CNN
-F 2 "Resistor_THT:R_Axial_DIN0922_L20.0mm_D9.0mm_P7.62mm_Vertical" H 5100 1300 50  0001 C CNN
+F 2 "Connector_JST:JST_EH_B2B-EH-A_1x02_P2.50mm_Vertical" H 5100 1300 50  0001 C CNN
 F 3 "~" H 5100 1300 50  0001 C CNN
 	1    5100 1300
@@
 F 0 "J1" H 928 1726 50  0000 L CNN
 F 1 "Conn_01x03_Female" H 928 1635 50  0000 L CNN
-F 2 "Connector_JST:JST_EH_B3B-EH-A_1x03_P2.50mm_Vertical" H 900 1700 50  0001 C CNN
+F 2 "Connector_JST:JST_NV_B03P-NV_1x03_P5.00mm_Vertical" H 900 1700 50  0001 C CNN
 F 3 "~" H 900 1700 50  0001 C CNN
 	1    900  1700

Commit message: Resistors changed and all paths routed
Parts:
- R10, R11, R12, R13, R2, R3, R4, R5, R6, R7, R8, R9: footprint Resistor_THT:R_Axial_DIN0207_L6.3mm_D2.5mm_P10.16mm_Horizontal -> Resistor_SMD:R_0805_2012Metric_Pad1.20x1.40mm_HandSolder
Changed lines of the file:
@@
 F 0 "R3" V 2243 3500 50  0000 C CNN
 F 1 "R" V 2334 3500 50  0000 C CNN
-F 2 "Resistor_THT:R_Axial_DIN0207_L6.3mm_D2.5mm_P10.16mm_Horizontal" V 2380 3500 50  0001 C CNN
+F 2 "Resistor_SMD:R_0805_2012Metric_Pad1.20x1.40mm_HandSolder" V 2380 3500 50  0001 C CNN
 F 3 "~" H 2450 3500 50  0001 C CNN
 	1    2450 3500
@@
 F 0 "R7" H 3170 3696 50  0000 L CNN
 F 1 "R" H 3170 3605 50  0000 L CNN
-F 2 "Resistor_THT:R_Axial_DIN0207_L6.3mm_D2.5mm_P10.16mm_Horizontal" V 3030 3650 50  0001 C CNN
+F 2 "Resistor_SMD:R_0805_2012Metric_Pad1.20x1.40mm_HandSolder" V 3030 3650 50  0001 C CNN
 F 3 "~" H 3100 3650 50  0001 C CNN
 	1    3100 3650
@@
 F 0 "R2" V 2193 4350 50  0000 C CNN
 F 1 "R" V 2284 4350 50  0000 C CNN
-F 2 "Resistor_THT:R_Axial_DIN0207_L6.3mm_D2.5mm_P10.16mm_Horizontal" V 2330 4350 50  0001 C CNN
+F 2 "Resistor_SMD:R_0805_2012Metric_Pad1.20x1.40mm_HandSolder" V 2330 4350 50  0001 C CNN
 F 3 "~" H 2400 4350 50  0001 C CNN
 	1    2400 4350
@@
 F 0 "R6" H 3120 4546 50  0000 L CNN
 F 1 "R" H 3120 4455 50  0000 L CNN
-F 2 "Resistor_THT:R_Axial_DIN0207_L6.3mm_D2.5mm_P10.16mm_Horizontal" V 2980 4500 50  0001 C CNN
+F 2 "Resistor_SMD:R_0805_2012Metric_Pad1.20x1.40mm_HandSolder" V 2980 4500 50  0001 C CNN
 F 3 "~" H 3050 4500 50  0001 C CNN
 	1    3050 4500
@@
 F 0 "R8" H 3170 7146 50  0000 L CNN
 F 1 "R" H 3170 7055 50  0000 L CNN
-F 2 "Resistor_THT:R_Axial_DIN0207_L6.3mm_D2.5mm_P10.16mm_Horizontal" V 3030 7100 50  0001 C CNN
+F 2 "Resistor_SMD:R_0805_2012Metric_Pad1.20x1.40mm_HandSolder" V 3030 7100 50  0001 C CNN
 F 3 "~" H 3100 7100 50  0001 C CNN
 	1    3100 7100
@@
 F 0 "R4" V 2243 6950 50  0000 C CNN
 F 1 "R" V 2334 6950 50  0000 C CNN
-F 2 "Resistor_THT:R_Axial_DIN0207_L6.3mm_D2.5mm_P10.16mm_Horizontal" V 2380 6950 50  0001 C CNN
+F 2 "Resistor_SMD:R_0805_2012Metric_Pad1.20x1.40mm_HandSolder" V 2380 6950 50  0001 C CNN
 F 3 "~" H 2450 6950 50  0001 C CNN
 	1    2450 6950
@@
 F 0 "R9" H 3220 6296 50  0000 L CNN
 F 1 "R" H 3220 6205 50  0000 L CNN
-F 2 "Resistor_THT:R_Axial_DIN0207_L6.3mm_D2.5mm_P10.16mm_Horizontal" V 3080 6250 50  0001 C CNN
+F 2 "Resistor_SMD:R_0805_2012Metric_Pad1.20x1.40mm_HandSolder" V 3080 6250 50  0001 C CNN
 F 3 "~" H 3150 6250 50  0001 C CNN
 	1    3150 6250
@@
 F 0 "R5" V 2293 6100 50  0000 C CNN
 F 1 "R" V 2384 6100 50  0000 C CNN
-F 2 "Resistor_THT:R_Axial_DIN0207_L6.3mm_D2.5mm_P10.16mm_Horizontal" V 2430 6100 50  0001 C CNN
+F 2 "Resistor_SMD:R_0805_2012Metric_Pad1.20x1.40mm_HandSolder" V 2430 6100 50  0001 C CNN
 F 3 "~" H 2500 6100 50  0001 C CNN
 	1    2500 6100
@@
 F 0 "R12" H 6370 7346 50  0000 L CNN
 F 1 "R" H 6370 7255 50  0000 L CNN
-F 2 "Resistor_THT:R_Axial_DIN0207_L6.3mm_D2.5mm_P10.16mm_Horizontal" V 6230 7300 50  0001 C CNN
+F 2 "Resistor_SMD:R_0805_2012Metric_Pad1.20x1.40mm_HandSolder" V 6230 7300 50  0001 C CNN
 F 3 "~" H 6300 7300 50  0001 C CNN
 	1    6300 7300
@@
 F 0 "R10" V 5443 7150 50  0000 C CNN
 F 1 "R" V 5534 7150 50  0000 C CNN
-F 2 "Resistor_THT:R_Axial_DIN0207_L6.3mm_D2.5mm_P10.16mm_Horizontal" V 5580 7150 50  0001 C CNN
+F 2 "Resistor_SMD:R_0805_2012Metric_Pad1.20x1.40mm_HandSolder" V 5580 7150 50  0001 C CNN
 F 3 "~" H 5650 7150 50  0001 C CNN
 	1    5650 7150
@@
 F 0 "R13" H 6420 6496 50  0000 L CNN
 F 1 "R" H 6420 6405 50  0000 L CNN
-F 2 "Resistor_THT:R_Axial_DIN0207_L6.3mm_D2.5mm_P10.16mm_Horizontal" V 6280 6450 50  0001 C CNN
+F 2 "Resistor_SMD:R_0805_2012Metric_Pad1.20x1.40mm_HandSolder" V 6280 6450 50  0001 C CNN
 F 3 "~" H 6350 6450 50  0001 C CNN
 	1    6350 6450
@@
 F 0 "R11" V 5493 6300 50  0000 C CNN
 F 1 "R" V 5584 6300 50  0000 C CNN
-F 2 "Resistor_THT:R_Axial_DIN0207_L6.3mm_D2.5mm_P10.16mm_Horizontal" V 5630 6300 50  0001 C CNN
+F 2 "Resistor_SMD:R_0805_2012Metric_Pad1.20x1.40mm_HandSolder" V 5630 6300 50  0001 C CNN
 F 3 "~" H 5700 6300 50  0001 C CNN
 	1    5700 6300
