File: WBC_transmitter/file5FEBA210.sch (KiCad schematic (older format))
At the start: 34 parts, among them U5 TL082

Commit message: Resistors changed and all paths routed
Parts:
- R14, R15, R16, R17, R18, R19, R20, R21, R22, R23, R24, R25, R26, R27, R28, R29, R30, R31, R32, R33, R34, R35: footprint Resistor_THT:R_Axial_DIN0207_L6.3mm_D2.5mm_P10.16mm_Horizontal -> Resistor_SMD:R_0805_2012Metric_Pad1.20x1.40mm_HandSolder
Changed lines of the file:
@@
 F 0 "R16" V 1243 2000 50  0000 C CNN
 F 1 "475k" V 1334 2000 50  0000 C CNN
-F 2 "Resistor_THT:R_Axial_DIN0207_L6.3mm_D2.5mm_P10.16mm_Horizontal" V 1380 2000 50  0001 C CNN
+F 2 "Resistor_SMD:R_0805_2012Metric_Pad1.20x1.40mm_HandSolder" V 1380 2000 50  0001 C CNN
 F 3 "~" H 1450 2000 50  0001 C CNN
 	1    1450 2000
@@
 F 0 "R20" V 1693 2000 50  0000 C CNN
 F 1 "475k" V 1784 2000 50  0000 C CNN
-F 2 "Resistor_THT:R_Axial_DIN0207_L6.3mm_D2.5mm_P10.16mm_Horizontal" V 1830 2000 50  0001 C CNN
+F 2 "Resistor_SMD:R_0805_2012Metric_Pad1.20x1.40mm_HandSolder" V 1830 2000 50  0001 C CNN
 F 3 "~" H 1900 2000 50  0001 C CNN
 	1    1900 2000
@@
 F 0 "R24" V 2143 2000 50  0000 C CNN
 F 1 "475k" V 2234 2000 50  0000 C CNN
-F 2 "Resistor_THT:R_Axial_DIN0207_L6.3mm_D2.5mm_P10.16mm_Horizontal" V 2280 2000 50  0001 C CNN
+F 2 "Resistor_SMD:R_0805_2012Metric_Pad1.20x1.40mm_HandSolder" V 2280 2000 50  0001 C CNN
 F 3 "~" H 2350 2000 50  0001 C CNN
 	1    2350 2000
@@
 F 0 "R28" V 2593 2000 50  0000 C CNN
 F 1 "475k" V 2684 2000 50  0000 C CNN
-F 2 "Resistor_THT:R_Axial_DIN0207_L6.3mm_D2.5mm_P10.16mm_Horizontal" V 2730 2000 50  0001 C CNN
+F 2 "Resistor_SMD:R_0805_2012Metric_Pad1.20x1.40mm_HandSolder" V 2730 2000 50  0001 C CNN
 F 3 "~" H 2800 2000 50  0001 C CNN
 	1    2800 2000
@@
 F 0 "R17" V 1243 2300 50  0000 C CNN
 F 1 "475k" V 1334 2300 50  0000 C CNN
-F 2 "Resistor_THT:R_Axial_DIN0207_L6.3mm_D2.5mm_P10.16mm_Horizontal" V 1380 2300 50  0001 C CNN
+F 2 "Resistor_SMD:R_0805_2012Metric_Pad1.20x1.40mm_HandSolder" V 1380 2300 50  0001 C CNN
 F 3 "~" H 1450 2300 50  0001 C CNN
 	1    1450 2300
@@
 F 0 "R21" V 1693 2300 50  0000 C CNN
 F 1 "475k" V 1784 2300 50  0000 C CNN
-F 2 "Resistor_THT:R_Axial_DIN0207_L6.3mm_D2.5mm_P10.16mm_Horizontal" V 1830 2300 50  0001 C CNN
+F 2 "Resistor_SMD:R_0805_2012Metric_Pad1.20x1.40mm_HandSolder" V 1830 2300 50  0001 C CNN
 F 3 "~" H 1900 2300 50  0001 C CNN
 	1    1900 2300
@@
 F 0 "R25" V 2143 2300 50  0000 C CNN
 F 1 "475k" V 2234 2300 50  0000 C CNN
-F 2 "Resistor_THT:R_Axial_DIN0207_L6.3mm_D2.5mm_P10.16mm_Horizontal" V 2280 2300 50  0001 C CNN
+F 2 "Resistor_SMD:R_0805_2012Metric_Pad1.20x1.40mm_HandSolder" V 2280 2300 50  0001 C CNN
 F 3 "~" H 2350 2300 50  0001 C CNN
 	1    2350 2300
@@
 F 0 "R29" V 2593 2300 50  0000 C CNN
 F 1 "475k" V 2684 2300 50  0000 C CNN
-F 2 "Resistor_THT:R_Axial_DIN0207_L6.3mm_D2.5mm_P10.16mm_Horizontal" V 2730 2300 50  0001 C CNN
+F 2 "Resistor_SMD:R_0805_2012Metric_Pad1.20x1.40mm_HandSolder" V 2730 2300 50  0001 C CNN
 F 3 "~" H 2800 2300 50  0001 C CNN
 	1    2800 2300
@@
 F 0 "R31" H 3180 1654 50  0000 R CNN
 F 1 "7.5k" H 3180 1745 50  0000 R CNN
-F 2 "Resistor_THT:R_Axial_DIN0207_L6.3mm_D2.5mm_P10.16mm_Horizontal" V 3180 1700 50  0001 C CNN
+F 2 "Resistor_SMD:R_0805_2012Metric_Pad1.20x1.40mm_HandSolder" V 3180 1700 50  0001 C CNN
 F 3 "~" H 3250 1700 50  0001 C CNN
 	1    3250 1700
@@
 F 0 "R33" V 3393 2450 50  0000 C CNN
 F 1 "7.5k" V 3484 2450 50  0000 C CNN
-F 2 "Resistor_THT:R_Axial_DIN0207_L6.3mm_D2.5mm_P10.16mm_Horizontal" V 3530 2450 50  0001 C CNN
+F 2 "Resistor_SMD:R_0805_2012Metric_Pad1.20x1.40mm_HandSolder" V 3530 2450 50  0001 C CNN
 F 3 "~" H 3600 2450 50  0001 C CNN
 	1    3600 2450
@@
 F 0 "R35" V 3793 2100 50  0000 C CNN
 F 1 "100" V 3884 2100 50  0000 C CNN
-F 2 "Resistor_THT:R_Axial_DIN0207_L6.3mm_D2.5mm_P10.16mm_Horizontal" V 3930 2100 50  0001 C CNN
+F 2 "Resistor_SMD:R_0805_2012Metric_Pad1.20x1.40mm_HandSolder" V 3930 2100 50  0001 C CNN
 F 3 "~" H 4000 2100 50  0001 C CNN
 	1    4000 2100
@@
 F 0 "R14" V 1193 4350 50  0000 C CNN
 F 1 "475k" V 1284 4350 50  0000 C CNN
-F 2 "Resistor_THT:R_Axial_DIN0207_L6.3mm_D2.5mm_P10.16mm_Horizontal" V 1330 4350 50  0001 C CNN
+F 2 "Resistor_SMD:R_0805_2012Metric_Pad1.20x1.40mm_HandSolder" V 1330 4350 50  0001 C CNN
 F 3 "~" H 1400 4350 50  0001 C CNN
 	1    1400 4350
@@
 F 0 "R18" V 1643 4350 50  0000 C CNN
 F 1 "475k" V 1734 4350 50  0000 C CNN
-F 2 "Resistor_THT:R_Axial_DIN0207_L6.3mm_D2.5mm_P10.16mm_Horizontal" V 1780 4350 50  0001 C CNN
+F 2 "Resistor_SMD:R_0805_2012Metric_Pad1.20x1.40mm_HandSolder" V 1780 4350 50  0001 C CNN
 F 3 "~" H 1850 4350 50  0001 C CNN
 	1    1850 4350
@@
 F 0 "R22" V 2093 4350 50  0000 C CNN
 F 1 "475k" V 2184 4350 50  0000 C CNN
-F 2 "Resistor_THT:R_Axial_DIN0207_L6.3mm_D2.5mm_P10.16mm_Horizontal" V 2230 4350 50  0001 C CNN
+F 2 "Resistor_SMD:R_0805_2012Metric_Pad1.20x1.40mm_HandSolder" V 2230 4350 50  0001 C CNN
 F 3 "~" H 2300 4350 50  0001 C CNN
 	1    2300 4350
@@
 F 0 "R26" V 2543 4350 50  0000 C CNN
 F 1 "475k" V 2634 4350 50  0000 C CNN
-F 2 "Resistor_THT:R_Axial_DIN0207_L6.3mm_D2.5mm_P10.16mm_Horizontal" V 2680 4350 50  0001 C CNN
+F 2 "Resistor_SMD:R_0805_2012Metric_Pad1.20x1.40mm_HandSolder" V 2680 4350 50  0001 C CNN
 F 3 "~" H 2750 4350 50  0001 C CNN
 	1    2750 4350
@@
 F 0 "R15" V 1193 4650 50  0000 C CNN
 F 1 "475k" V 1284 4650 50  0000 C CNN
-F 2 "Resistor_THT:R_Axial_DIN0207_L6.3mm_D2.5mm_P10.16mm_Horizontal" V 1330 4650 50  0001 C CNN
+F 2 "Resistor_SMD:R_0805_2012Metric_Pad1.20x1.40mm_HandSolder" V 1330 4650 50  0001 C CNN
 F 3 "~" H 1400 4650 50  0001 C CNN
 	1    1400 4650
@@
 F 0 "R19" V 1643 4650 50  0000 C CNN
 F 1 "475k" V 1734 4650 50  0000 C CNN
-F 2 "Resistor_THT:R_Axial_DIN0207_L6.3mm_D2.5mm_P10.16mm_Horizontal" V 1780 4650 50  0001 C CNN
+F 2 "Resistor_SMD:R_0805_2012Metric_Pad1.20x1.40mm_HandSolder" V 1780 4650 50  0001 C CNN
 F 3 "~" H 1850 4650 50  0001 C CNN
 	1    1850 4650
@@
 F 0 "R23" V 2093 4650 50  0000 C CNN
 F 1 "475k" V 2184 4650 50  0000 C CNN
-F 2 "Resistor_THT:R_Axial_DIN0207_L6.3mm_D2.5mm_P10.16mm_Horizontal" V 2230 4650 50  0001 C CNN
+F 2 "Resistor_SMD:R_0805_2012Metric_Pad1.20x1.40mm_HandSolder" V 2230 4650 50  0001 C CNN
 F 3 "~" H 2300 4650 50  0001 C CNN
 	1    2300 4650
@@
 F 0 "R27" V 2543 4650 50  0000 C CNN
 F 1 "475k" V 2634 4650 50  0000 C CNN
-F 2 "Resistor_THT:R_Axial_DIN0207_L6.3mm_D2.5mm_P10.16mm_Horizontal" V 2680 4650 50  0001 C CNN
+F 2 "Resistor_SMD:R_0805_2012Metric_Pad1.20x1.40mm_HandSolder" V 2680 4650 50  0001 C CNN
 F 3 "~" H 2750 4650 50  0001 C CNN
 	1    2750 4650
@@
 F 0 "R30" H 3130 4004 50  0000 R CNN
 F 1 "7.5k" H 3130 4095 50  0000 R CNN
-F 2 "Resistor_THT:R_Axial_DIN0207_L6.3mm_D2.5mm_P10.16mm_Horizontal" V 3130 4050 50  0001 C CNN
+F 2 "Resistor_SMD:R_0805_2012Metric_Pad1.20x1.40mm_HandSolder" V 3130 4050 50  0001 C CNN
 F 3 "~" H 3200 4050 50  0001 C CNN
 	1    3200 4050
@@
 F 0 "R32" V 3343 4800 50  0000 C CNN
 F 1 "7.5k" V 3434 4800 50  0000 C CNN
-F 2 "Resistor_THT:R_Axial_DIN0207_L6.3mm_D2.5mm_P10.16mm_Horizontal" V 3480 4800 50  0001 C CNN
+F 2 "Resistor_SMD:R_0805_2012Metric_Pad1.20x1.40mm_HandSolder" V 3480 4800 50  0001 C CNN
 F 3 "~" H 3550 4800 50  0001 C CNN
 	1    3550 4800
@@
 F 0 "R34" V 3743 4450 50  0000 C CNN
 F 1 "100" V 3834 4450 50  0000 C CNN
-F 2 "Resistor_THT:R_Axial_DIN0207_L6.3mm_D2.5mm_P10.16mm_Horizontal" V 3880 4450 50  0001 C CNN
+F 2 "Resistor_SMD:R_0805_2012Metric_Pad1.20x1.40mm_HandSolder" V 3880 4450 50  0001 C CNN
 F 3 "~" H 3950 4450 50  0001 C CNN
 	1    3950 4450
